Commit message: minor changes

File: custom_bot/urdf/robot.urdf (robot description, URDF)
Before this commit: robot diffbot, 6 links, 5 joints
Links:
- added link caster_wheel2, mass 0.25; collision sphere radius=0.05; visual sphere radius=0.05
Joints:
- added joint caster_wheel_joint2: type fixed, parent base_link, child caster_wheel2, origin xyz=-0.2 0 -0.1, axis 0 0 1
